File: Fader/MHCI-Fader/MHCI-Fader.kicad_pcb (KiCad board)
At the start: 2 copper layers, 107.5 x 20 mm, 31 parts, among them J1 Conn_01x06, SW1 SW_Push_LED, U3 SRV05-4, U4 TXB0102DCU, U5 TJA1051T-3

Commit message: Logos and description
Routing:
- net GND: vias 58 -> 52
Other:
- board text added: "MHCI Fader Control v1.0"
Changed lines of the file:
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@@
 		(layer "B.SilkS")
+	)
+	(gr_poly
+		(pts
+			(xy 138.871244 106.68) (xy 137.561246 107.120002) (xy 137.561245 107.230002) (xy 138.871244 107.67)
+			(xy 138.871246 107.440002) (xy 138.001247 107.180002) (xy 138.871244 106.910002)
+		)
+		(stroke
+			(width 0.05)
+			(type solid)
+		)
+		(fill solid)
+		(layer "F.SilkS")
 	)
 	(gr_line
@@
 			(polygon
 				(pts
-					(xy 117.146999 111.6225) (xy 117.146999 110.51095) (xy 117.500174 110.51095) (xy 117.500174 110.30945)
-					(xy 116.545795 110.30945) (xy 116.545795 110.51095) (xy 116.917288 110.51095) (xy 116.917288 111.6225)
+					(xy 117.146266 111.6225) (xy 117.146266 110.509851) (xy 117.500906 110.509851) (xy 117.500906 110.30945)
+					(xy 116.544696 110.30945) (xy 116.544696 110.509851) (xy 116.918387 110.509851) (xy 116.918387 111.6225)
 				)
 			)
 			(polygon
 				(pts
-					(xy 116.097731 111.6225) (xy 116.097731 110.51095) (xy 116.450906 110.51095) (xy 116.450906 110.30945)
-					(xy 115.496527 110.30945) (xy 115.496527 110.51095) (xy 115.868021 110.51095) (xy 115.868021 111.6225)
+					(xy 116.096999 111.6225) (xy 116.096999 110.509851) (xy 116.451639 110.509851) (xy 116.451639 110.30945)
+					(xy 115.495428 110.30945) (xy 115.495428 110.509851) (xy 115.86912 110.509851) (xy 115.86912 111.6225)
 				)
 			)
@@
 		)
 	)
+	(gr_text "MHCI\nFader Control\nv1.0"
+		(at 143.971244 107.880001 90)
+		(layer "F.SilkS")
+		(effects
+			(font
+				(size 1 1)
+				(thickness 0.15)
+			)
+			(justify left bottom)
+		)
+	)
 	(gr_text "L"
 		(at 74.8 105.6 90)
@@
 		)
 	)
-	(gr_text "Followspot\nFader\nV1.0"
-		(at 142.75 102 90)
+	(gr_text "TT"
+		(at 138.261247 105.590002 90)
 		(layer "F.SilkS")
 		(effects
 			(font
-				(size 1 1)
-				(thickness 0.15)
+				(face "Inconsolata")
+				(size 1.5 1.5)
+				(thickness 0.3)
+				(bold yes)
 			)
-			(justify bottom)
+		)
+		(render_cache "TT" 90
+			(polygon
+				(pts
+					(xy 138.883747 106.236268) (xy 137.771098 106.236268) (xy 137.771098 106.590908) (xy 137.570697 106.590908)
+					(xy 137.570697 105.634698) (xy 137.771098 105.634698) (xy 137.771098 106.008389) (xy 138.883747 106.008389)
+				)
+			)
+			(polygon
+				(pts
+					(xy 138.883747 105.187001) (xy 137.771098 105.187001) (xy 137.771098 105.541641) (xy 137.570697 105.541641)
+					(xy 137.570697 104.58543) (xy 137.771098 104.58543) (xy 137.771098 104.959122) (xy 138.883747 104.959122)
+				)
+			)
 		)
 	)
@@
 	)
 	(via
-		(at 143 101)
-		(size 0.9)
-		(drill 0.4)
-		(layers "F.Cu" "B.Cu")
-		(free yes)
-		(net 32)
-	)
-	(via
 		(at 97 94)
 		(size 0.9)
@@
 	)
 	(via
-		(at 137 105)
-		(size 0.9)
-		(drill 0.4)
-		(layers "F.Cu" "B.Cu")
-		(free yes)
-		(net 32)
-	)
-	(via
 		(at 115 102)
 		(size 0.9)
@@
 	)
 	(via
-		(at 143 98)
-		(size 0.9)
-		(drill 0.4)
-		(layers "F.Cu" "B.Cu")
-		(free yes)
-		(net 32)
-	)
-	(via
-		(at 143 105)
-		(size 0.9)
-		(drill 0.4)
-		(layers "F.Cu" "B.Cu")
-		(free yes)
-		(net 32)
-	)
-	(via
 		(at 100 96)
 		(size 0.9)
@@
 	)
 	(via
-		(at 140 103)
-		(size 0.9)
-		(drill 0.4)
-		(layers "F.Cu" "B.Cu")
-		(free yes)
-		(net 32)
-	)
-	(via
 		(at 146 103)
 		(size 0.9)
@@
 		(size 0.9)
 		(drill 0.4)
-		(layers "F.Cu" "B.Cu")
-		(free yes)
-		(net 32)
-	)
-	(via
-		(at 140 96)
-		(size 0.9)
-		(drill 0.4)

Commit message: MHCI Production Read
Other:
- board text removed: "TOOLING HOLES MOUNTING HOLES"
Changed lines of the file:
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@@
 	(gr_poly
 		(pts
-			(xy 138.871244 106.68) (xy 137.561246 107.120002) (xy 137.561245 107.230002) (xy 138.871244 107.67)
-			(xy 138.871246 107.440002) (xy 138.001247 107.180002) (xy 138.871244 106.910002)
+			(xy 138.869997 105.899998) (xy 137.559999 106.34) (xy 137.559998 106.45) (xy 138.869997 106.889998)
+			(xy 138.869999 106.66) (xy 138 106.4) (xy 138.869997 106.13)
 		)
 		(stroke
@@
 	)
 	(gr_text "MHCI\nFader Control\nv1.0"
-		(at 143.971244 107.880001 90)
+		(at 143.969997 107.099999 90)
 		(layer "F.SilkS")
 		(effects
@@
 	)
 	(gr_text "TT"
-		(at 138.261247 105.590002 90)
+		(at 138.26 104.81 90)
 		(layer "F.SilkS")
 		(effects
@@
 			(polygon
 				(pts
-					(xy 138.883747 106.236268) (xy 137.771098 106.236268) (xy 137.771098 106.590908) (xy 137.570697 106.590908)
-					(xy 137.570697 105.634698) (xy 137.771098 105.634698) (xy 137.771098 106.008389) (xy 138.883747 106.008389)
+					(xy 138.8825 105.456266) (xy 137.769851 105.456266) (xy 137.769851 105.810906) (xy 137.56945 105.810906)
+					(xy 137.56945 104.854696) (xy 137.769851 104.854696) (xy 137.769851 105.228387) (xy 138.8825 105.228387)
 				)
 			)
 			(polygon
 				(pts
-					(xy 138.883747 105.187001) (xy 137.771098 105.187001) (xy 137.771098 105.541641) (xy 137.570697 105.541641)
-					(xy 137.570697 104.58543) (xy 137.771098 104.58543) (xy 137.771098 104.959122) (xy 138.883747 104.959122)
+					(xy 138.8825 104.406999) (xy 137.769851 104.406999) (xy 137.769851 104.761639) (xy 137.56945 104.761639)
+					(xy 137.56945 103.805428) (xy 137.769851 103.805428) (xy 137.769851 104.17912) (xy 138.8825 104.17912)
 				)
 			)
@@
 		)
 	)
-	(gr_text "TOOLING HOLES\nMOUNTING HOLES"
-		(at 102 123 0)
-		(layer "Dwgs.User")
-		(effects
-			(font
-				(size 3 3)
-				(thickness 0.6)
-				(bold yes)
-			)
-			(justify left bottom)
-		)
-	)
